Commit message: update odom

File: src/cpp01_urdf/urdf/urdf/CyberNaviRobot.urdf (robot description, URDF)
Before this commit: robot CyberNaviRobot, 5 links, 4 joints
Links:
- added link laser, mass 0.1; collision box size=0.05 0.05 0.05; visual box size=0.01 0.01 0.01
- added link odom
Joints:
- added joint laser_joint: type fixed, parent base_link, child laser, origin xyz=0.05 0 0.235 rpy=0 0 0
- added joint odom_joint: type fixed, parent odom, child base_link, origin xyz=0 0 0 rpy=0 0 0
